Commit message: feat(perception): add 2D YOLOv8 perception pipeline, OAK-D sensor integration, and 3D simulation setup

File: src/terrascout_description/urdf/scout.urdf.xacro (robot description, xacro)
@@ -200,4 +200,46 @@
     </sensor>
   </gazebo>
+  <material name="black">
+    <color rgba="0.1 0.1 0.1 1.0"/>
+  </material>
+  <joint name="oakd_joint" type="fixed">
+    <parent link="base_link"/>
+    <child link="oakd_link"/>
+    <origin xyz="0.36 0 0.22" rpy="0 0 0"/>
+  </joint>
+  <link name="oakd_link">
+    <visual>
+      <geometry>
+        <box size="0.0229 0.097 0.0295"/>
+      </geometry>
+      <material name="black"/>
+    </visual>
+  </link>
+  <joint name="oakd_rgb_optical_joint" type="fixed">
+    <parent link="oakd_link"/>
+    <child link="oakd_rgb_optical_frame"/>
+    <origin xyz="0 0 0" rpy="-1.5707963 0 -1.5707963"/>
+  </joint>
+  <link name="oakd_rgb_optical_frame"/>
+  <gazebo reference="oakd_link">
+    <sensor name="oakd_rgbd_sensor" type="rgbd_camera">
+      <always_on>true</always_on>
+      <update_rate>30</update_rate>
+      <topic>${ns}/oakd</topic>
+      <gz_frame_id>oakd_rgb_optical_frame</gz_frame_id>
+      <camera>
+        <horizontal_fov>1.43</horizontal_fov>
+        <image>
+          <width>1280</width>
+          <height>720</height>
+          <format>R8G8B8</format>
+        </image>
+        <clip>
+          <near>0.2</near>
+          <far>15.0</far>
+        </clip>
+      </camera>
+    </sensor>
+  </gazebo>
   <joint name="navsat_joint" type="fixed">
     <parent link="base_link"/>
